Commit message: v1.4.3

File: include/ur5.urdf (robot description, URDF)
Before this commit: robot ur5, 13 links, 12 joints
Joints:
- joint flange-tool0: origin xyz=0 0 0 rpy=1.5707963267948966 0 1.5707963267948966 -> xyz=0 0 -0.5 rpy=1.5707963267948966 0 1.5707963267948966

Commit message: v1.4.4

File: include/ur5.urdf (robot description, URDF)
Before this commit: robot ur5, 13 links, 12 joints
Joints:
- joint flange-tool0: origin xyz=0 0 -0.5 rpy=1.5707963267948966 0 1.5707963267948966 -> xyz=0 0 0.5 rpy=1.5707963267948966 0 1.5707963267948966

Commit message: v3.7.0

File: include/ur5.urdf (robot description, URDF)
Before this commit: robot ur5, 13 links, 12 joints
Joints:
- joint flange-tool0: origin xyz=0 0 0.5 rpy=1.5707963267948966 0 1.5707963267948966 -> xyz=0.5 0 0 rpy=1.5707963267948966 0 1.5707963267948966

File: urdf/ur_macro.xacro (robot description, xacro)
@@ -440,5 +440,5 @@
     <joint name="${tf_prefix}flange-tool0" type="fixed">
       <!-- default toolframe - X+ left, Y+ up, Z+ front -->
-      <origin xyz="0 0 0" rpy="${pi/2.0} 0 ${pi/2.0}"/>
+      <origin xyz="0.5 0 0.0" rpy="${pi/2.0} 0 ${pi/2.0}"/>
       <parent link="${tf_prefix}flange"/>
       <child link="${tf_prefix}tool0"/>
