Commit message: v5.4

File: ur5_simulation/include/ur5.urdf (robot description, URDF)
Before this commit: robot ur5, 13 links, 12 joints
Joints:
- joint flange-tool0: origin xyz=0.5 0 0 rpy=1.5707963267948966 0 1.5707963267948966 -> xyz=0.5 0 -0.05 rpy=1.5707963267948966 0 1.5707963267948966

File: ur5_simulation/include/ur5e.urdf (robot description, URDF)
Before this commit: robot ur5e, 13 links, 12 joints
Joints:
- joint flange-tool0: origin xyz=0 0 0 rpy=1.5707963267948966 0 1.5707963267948966 -> xyz=0.5 0 -0.05 rpy=1.5707963267948966 0 1.5707963267948966

File: ur5_simulation/urdf/ur_macro.xacro (robot description, xacro)
@@ -440,5 +440,5 @@
     <joint name="${tf_prefix}flange-tool0" type="fixed">
       <!-- default toolframe - X+ left, Y+ up, Z+ front -->
-      <origin xyz="0.5 0 0.0" rpy="${pi/2.0} 0 ${pi/2.0}"/>
+      <origin xyz="0.5 0 -0.05" rpy="${pi/2.0} 0 ${pi/2.0}"/>
       <parent link="${tf_prefix}flange"/>
       <child link="${tf_prefix}tool0"/>

Commit message: v5.5.1

File: ur5_simulation/include/ur5.urdf (robot description, URDF)
Before this commit: robot ur5, 13 links, 12 joints
Joints:
- joint flange-tool0: origin xyz=0.5 0 -0.05 rpy=1.5707963267948966 0 1.5707963267948966 -> xyz=0.63 0 -0.05 rpy=1.5707963267948966 0 1.5707963267948966

File: ur5_simulation/include/ur5e.urdf (robot description, URDF)
Before this commit: robot ur5e, 13 links, 12 joints
Joints:
- joint flange-tool0: origin xyz=0.5 0 -0.05 rpy=1.5707963267948966 0 1.5707963267948966 -> xyz=0.63 0 -0.05 rpy=1.5707963267948966 0 1.5707963267948966

File: ur5_simulation/urdf/ur_macro.xacro (robot description, xacro)
@@ -440,5 +440,5 @@
     <joint name="${tf_prefix}flange-tool0" type="fixed">
       <!-- default toolframe - X+ left, Y+ up, Z+ front -->
-      <origin xyz="0.5 0 -0.05" rpy="${pi/2.0} 0 ${pi/2.0}"/>
+      <origin xyz="0.63 0 -0.05" rpy="${pi/2.0} 0 ${pi/2.0}"/>
       <parent link="${tf_prefix}flange"/>
       <child link="${tf_prefix}tool0"/>
