Commit message: v14.07 reforma interfaz

File: ur5e_bringup/urdf/tool.urdf.xacro (robot description, xacro)
@@ -32,8 +32,11 @@
         </geometry>
       </visual>
+      <!-- tool_collision.dae = tool.dae sin su bloque <lines> (12 aristas
+           sueltas, sin volumen): el detector de colisiones de Gazebo
+           (DART/ODE) asume solo triangulos y hace segfault con ellas. -->
       <collision>
         <origin xyz="0 ${-mesh_gap} 0" rpy="0 0 0"/>
         <geometry>
-          <mesh filename="package://ur5e_bringup/meshes/tool/tool.dae"/>
+          <mesh filename="package://ur5e_bringup/meshes/tool/tool_collision.dae"/>
         </geometry>
       </collision>

File: ur5e_bringup/urdf/ur5e_single.urdf.xacro (robot description, xacro)
@@ -19,4 +19,7 @@
   <xacro:arg name="robot_ip" default="0.0.0.0" />
   <xacro:arg name="use_fake_hardware" default="true" />
+  <!-- Gazebo (multi_ur5e_sim.launch.py); requiere use_fake_hardware:=false -->
+  <xacro:arg name="sim_ignition" default="false" />
+  <xacro:arg name="simulation_controllers" default="" />
   <xacro:arg name="headless_mode" default="true" />
   <xacro:arg name="reverse_port" default="50001" />
@@ -39,4 +42,6 @@
     robot_ip="$(arg robot_ip)"
     use_fake_hardware="$(arg use_fake_hardware)"
+    sim_ignition="$(arg sim_ignition)"
+    simulation_controllers="$(arg simulation_controllers)"
     headless_mode="$(arg headless_mode)"
     reverse_port="$(arg reverse_port)"

File: ur5e_bringup/urdf/ur5e_unit.xacro (robot description, xacro)
@@ -12,8 +12,15 @@
                   ur_description/config/<ur_type>/
     robot_ip    : IP del controlador real (ur_robot_driver). Ignorada si
-                  use_fake_hardware=true
+                  use_fake_hardware=true o sim_ignition=true
+    sim_ignition: simular en Gazebo (Ignition Fortress) con ign_ros2_control
+                  en vez del driver real / mock. Excluyente con
+                  use_fake_hardware (ambos meterian su plugin en <hardware>)
+    simulation_controllers : ruta del yaml de controladores que recibe el
+                  controller_manager que crea el plugin de Gazebo (solo se
+                  usa con sim_ignition=true)
   -->
   <xacro:include filename="$(find ur_description)/urdf/ur_macro.xacro" />
   <xacro:include filename="$(find ur5e_bringup)/urdf/tool.urdf.xacro" />
+  <xacro:include filename="$(find ur5e_bringup)/urdf/ur_sim.ros2_control.xacro" />
   <xacro:macro name="ur5e_unit" params="
       name
@@ -25,4 +32,6 @@
       robot_ip:=0.0.0.0
       use_fake_hardware:=true
+      sim_ignition:=false
+      simulation_controllers:=''
       headless_mode:=true
       safety_limits:=true
@@ -54,4 +63,5 @@
       safety_k_position="${safety_k_position}"
       use_fake_hardware="${use_fake_hardware}"
+      sim_ignition="${sim_ignition}"
       headless_mode="${headless_mode}"
       robot_ip="${robot_ip}"
@@ -62,7 +72,11 @@
       script_filename="to_be_filled_by_ur_robot_driver"
       output_recipe_filename="to_be_filled_by_ur_robot_driver"
-      input_recipe_filename="to_be_filled_by_ur_robot_driver">
+      input_recipe_filename="to_be_filled_by_ur_robot_driver"
+      generate_ros2_control_tag="${str(sim_ignition).lower() != 'true'}">
       <origin xyz="0 0 0" rpy="0 0 0" />
     </xacro:ur_robot>
+    <!-- En Gazebo el <ros2_control> lo arma ur_sim_ros2_control (abajo) en
+         vez de ur_description, para poder declarar el sensor F/T. -->
+    <xacro:property name="_is_sim" value="${str(sim_ignition).lower() == 'true'}" />
     <xacro:if value="${attach_tool}">
       <xacro:tool
@@ -72,4 +86,40 @@
         rpy="${tool_rpy}" />
     </xacro:if>
+    <!-- Gazebo: el plugin crea el controller_manager de ESTE robot dentro
+         del simulador, en el namespace /<name> (mismo que usa el launch),
+         y lee robot_description de /<name>/robot_state_publisher. -->
+    <xacro:if value="${_is_sim}">
+      <gazebo>
+        <plugin filename="libign_ros2_control-system.so"
+                name="ign_ros2_control::IgnitionROS2ControlPlugin">
+          <parameters>${simulation_controllers}</parameters>
+          <ros>
+            <namespace>/${name}</namespace>
+          </ros>
+        </plugin>
+      </gazebo>
+      <xacro:ur_sim_ros2_control name="${name}" tf_prefix="${tf_prefix}" />
+      <!-- Sensor F/T del TCP, como el del UR e-Series: en el joint
+           flange -> tool0, medido en el frame de tool0 (el driver real
+           publica la fuerza en el frame del TCP; con TCP nulo en el
+           pendant eso es tool0). child_to_parent = fuerza que el lado de la
+           herramienta ejerce sobre la brida: con la herramienta quieta es
+           la fuerza externa + su peso (como un payload sin compensar).
+           preserveFixedJoint: si no, Gazebo fusiona los joints fijos y el
+           sensor desaparece con el joint. Se llama igual que el <sensor>
+           de ur_sim_ros2_control, que es como IgnitionSystem lo asocia. -->
+      <gazebo reference="${tf_prefix}flange-tool0">
+        <preserveFixedJoint>true</preserveFixedJoint>
+        <sensor name="${tf_prefix}tcp_fts_sensor" type="force_torque">
+          <always_on>true</always_on>
+          <update_rate>500</update_rate>
+          <topic>/${name}/tcp_fts</topic>
+          <force_torque>
+            <frame>child</frame>
+            <measure_direction>child_to_parent</measure_direction>
+          </force_torque>
+        </sensor>
+      </gazebo>
+    </xacro:if>
   </xacro:macro>
 </robot>
